Commit message: added mujoco position and velocity interface and bringup to support all controllers in mujoco sim

File: src/robotarm_mujoco/urdf/robotarm_sim.ros2_control.xacro (robot description, xacro)
@@ -1,16 +1,21 @@
 <?xml version="1.0"?>
-<!-- ros2_control block of the MuJoCo simulation. Effort only: the sim stands in for the motors in torque mode,
-     position/velocity controllers stay on mock_components. Each joint is driven by the MJCF <motor> actuator of the
-     same name. The joint list duplicates robotarm_description/urdf/robotarm.ros2_control.xacro, test_mjcf.py checks
-     that both stay equal. No torque_ff (moteus only) and no transmissions: MuJoCo drives axis5/axis6 directly. -->
+<!-- ros2_control block of the MuJoCo simulation. Each joint is driven by the MJCF <motor> actuator of the same name:
+     effort goes to it directly, position and velocity through the sim PIDs of config/sim_pids.yaml (a generic PID,
+     not a model of the moteus position loop). Position wins when a controller claims position and velocity, see
+     robotarm_mujoco_hardware. The joint list duplicates robotarm_description/urdf/robotarm.ros2_control.xacro,
+     test_mjcf.py checks that both stay equal. No torque_ff (moteus only, it only improves tracking) and no
+     transmissions: MuJoCo drives axis5/axis6 directly. -->
 <robot xmlns:xacro="http://www.ros.org/wiki/xacro">
-  <xacro:macro name="robotarm_sim_ros2_control" params="name mujoco_model headless:=false">
+  <xacro:macro name="robotarm_sim_ros2_control" params="name mujoco_model pids_config_file headless:=false">
     <ros2_control name="${name}" type="system">
       <hardware>
-        <plugin>mujoco_ros2_control/MujocoSystemInterface</plugin>
+        <plugin>robotarm_mujoco_hardware/RobotarmMujocoSystem</plugin>
         <param name="mujoco_model">${mujoco_model}</param>
         <param name="headless">${str(headless).lower()}</param>
+        <param name="pids_config_file">${pids_config_file}</param>
       </hardware>
       <joint name="axis1">
+        <command_interface name="position"/>
+        <command_interface name="velocity"/>
         <command_interface name="effort"/>
         <state_interface name="position"/>
@@ -19,4 +24,6 @@
       </joint>
       <joint name="axis2">
+        <command_interface name="position"/>
+        <command_interface name="velocity"/>
         <command_interface name="effort"/>
         <state_interface name="position"/>
@@ -25,4 +32,6 @@
       </joint>
       <joint name="axis3">
+        <command_interface name="position"/>
+        <command_interface name="velocity"/>
         <command_interface name="effort"/>
         <state_interface name="position"/>
@@ -31,4 +40,6 @@
       </joint>
       <joint name="axis4">
+        <command_interface name="position"/>
+        <command_interface name="velocity"/>
         <command_interface name="effort"/>
         <state_interface name="position"/>
@@ -37,4 +48,6 @@
       </joint>
       <joint name="axis5">
+        <command_interface name="position"/>
+        <command_interface name="velocity"/>
         <command_interface name="effort"/>
         <state_interface name="position"/>
@@ -43,4 +56,6 @@
       </joint>
       <joint name="axis6">
+        <command_interface name="position"/>
+        <command_interface name="velocity"/>
         <command_interface name="effort"/>
         <state_interface name="position"/>

File: src/robotarm_mujoco/urdf/robotarm_sim.urdf.xacro (robot description, xacro)
@@ -9,11 +9,15 @@
   <xacro:arg name="mujoco_model" default="" />
   <xacro:arg name="headless" default="false" />
+  <!-- position/velocity PID gains of the sim, empty: the installed config/sim_pids.yaml -->
+  <xacro:arg name="pids_config_file" default="" />
   <xacro:include filename="$(find robotarm_description)/urdf/robotarm_geometry.xacro" />
   <xacro:include filename="$(find robotarm_description)/urdf/tools/$(arg tool).xacro" />
   <xacro:include filename="$(find robotarm_mujoco)/urdf/robotarm_sim.ros2_control.xacro" />
+  <xacro:property name="default_pids" value="$(find robotarm_mujoco)/config/sim_pids.yaml" />
   <xacro:robotarm_geometry />
   <xacro:tool parent="flange" />
   <!-- same component name as the real hardware, so robotarm_bringup's controllers.yaml applies unchanged -->
   <xacro:robotarm_sim_ros2_control name="moteus_hardware_system"
-      mujoco_model="$(arg mujoco_model)" headless="$(arg headless)" />
+      mujoco_model="$(arg mujoco_model)" headless="$(arg headless)"
+      pids_config_file="${default_pids if '$(arg pids_config_file)' == '' else '$(arg pids_config_file)'}" />
 </robot>
